File: pcb/LNA/LNA.kicad_sch (KiCad schematic)
At the start: 0 parts

Commit message: Finished routing with 0805 components
Parts:
- added C1, C2, C3, C4, C5: C_0805, PCM_Capacitor_SMD_AKL:C_0805_2012Metric, symbol PCM_Capacitor_AKL:C_0805
- added J1, J2: SMA_Edge, PCM_SparkFun-Connector:SMA_Edge_8mm, symbol PCM_SparkFun-RF:SMA_EdgeMount_8mm
- added J3: Socket_01x02, Connector_PinHeader_2.54mm:PinHeader_2x01_P2.54mm_Vertical, symbol PCM_4ms_Connector:Socket_01x02
- added L2, L3: L_0805, PCM_SparkFun-Coil:0805, symbol Device:L
- added Q1: BFP460, PCM_Package_TO_SOT_SMD_AKL:SOT-343_SC-70-4, symbol PCM_Transistor_BJT_AKL:BFP450
- added R1, R2, R3: R_0805, PCM_Resistor_SMD_AKL:R_0805_2012Metric, symbol PCM_Resistor_US_AKL:R_0805
Connections:
- new net: C5.2, J1.1 (In), L3.2
- new net: C3.1, C4.1, L2.2
- new net: C2.1, Q1.3 (C), R1.1, R2.2
- new net: C3.2, Q1.1 (B), R1.2
- new net: J2.1 (In), L2.1
- new net: C2.2, L3.1
- new net 5V: J3.1 (Pin_1), R2.1
- new net EMITTER: C1.1, Q1.2 (E), Q1.4 (E), R3.1
- new net GND: C1.2, C4.2, C5.1, J1.2 (Ext), J2.2 (Ext), J3.2 (Pin_2), R3.2
